File: schematic/water-sensor.sch (EAGLE design)
At the start: 8 parts, among them X1 XRJK-S-01-6-4-0-9M2

Commit message: water sensor
Parts:
- removed X1: XRJK-S-01-6-4-0-9M2, con-xmultiple:XRJK-S-01-6-4-0-9M2
- added X2: 14867, con-4ucon:14867
Connections:
- net 5V: now also U$2.VCC
- net D10: now also U$2.CS
- net D11: now also U$2.SI
- net D12: now also U$2.SO
- net D13: now also U$2.SCK
- net D2: now also U$2.INT
- net GND: now also U$2.GND, X2.2
- net RESET: now also U$2.RESET
- net VIN: now also X2.1
Changed lines of the file:
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@@
 <part name="U$1" library="CRE-Lib1" deviceset="ARDUINONANO" device=""/>
 <part name="U$2" library="enc28j60" deviceset="ENC28J60" device="ENC28J60"/>
-<part name="X1" library="con-xmultiple" deviceset="XRJK*4" device="-0-9M2" technology="-S-01-6-"/>
+<part name="X2" library="con-4ucon" deviceset="14867" device=""/>
 </parts>
 <sheets>
@@
 <instance part="U$1" gate="G$1" x="53.34" y="83.82"/>
 <instance part="U$2" gate="G$1" x="147.32" y="35.56"/>
-<instance part="X1" gate="G$1" x="144.78" y="91.44"/>
+<instance part="X2" gate="G$1" x="139.7" y="91.44"/>
 </instances>
 <busses>
@@
 <wire x1="78.74" y1="66.04" x2="91.44" y2="66.04" width="0.1524" layer="91"/>
 <label x="88.9" y="66.04" size="1.778" layer="95"/>
+</segment>
+<segment>
+<pinref part="U$2" gate="G$1" pin="VCC"/>
+<wire x1="149.86" y1="50.8" x2="162.56" y2="50.8" width="0.1524" layer="91"/>
 </segment>
 </net>
@@
 <wire x1="137.16" y1="93.98" x2="129.54" y2="93.98" width="0.1524" layer="91"/>
 <wire x1="129.54" y1="93.98" x2="129.54" y2="88.9" width="0.1524" layer="91"/>
+<pinref part="X2" gate="G$1" pin="2"/>
 </segment>
 <segment>
@@
 <label x="88.9" y="76.2" size="1.778" layer="95"/>
 </segment>
+<segment>
+<pinref part="U$2" gate="G$1" pin="GND"/>
+<wire x1="124.46" y1="50.8" x2="114.3" y2="50.8" width="0.1524" layer="91"/>
+</segment>
 </net>
 <net name="VIN" class="0">
@@
 <wire x1="129.54" y1="96.52" x2="129.54" y2="101.6" width="0.1524" layer="91"/>
 <label x="129.54" y="101.6" size="1.778" layer="95"/>
+<pinref part="X2" gate="G$1" pin="1"/>
 </segment>
 <segment>
@@
 <label x="88.9" y="71.12" size="1.778" layer="95"/>
 </segment>
+<segment>
+<pinref part="U$2" gate="G$1" pin="RESET"/>
+<wire x1="124.46" y1="45.72" x2="114.3" y2="45.72" width="0.1524" layer="91"/>
+</segment>
 </net>
 <net name="D2" class="0">
@@
 <wire x1="48.26" y1="60.96" x2="35.56" y2="60.96" width="0.1524" layer="91"/>
 <label x="35.56" y="60.96" size="1.778" layer="95"/>
+</segment>
+<segment>
+<pinref part="U$2" gate="G$1" pin="INT"/>
+<wire x1="124.46" y1="30.48" x2="114.3" y2="30.48" width="0.1524" layer="91"/>
 </segment>
 </net>
@@
 <label x="35.56" y="20.32" size="1.778" layer="95"/>
 </segment>
+<segment>
+<pinref part="U$2" gate="G$1" pin="CS"/>
+<wire x1="149.86" y1="45.72" x2="162.56" y2="45.72" width="0.1524" layer="91"/>
+</segment>
 </net>
 <net name="D11" class="0">
@@
 <wire x1="48.26" y1="15.24" x2="35.56" y2="15.24" width="0.1524" layer="91"/>
 <label x="35.56" y="15.24" size="1.778" layer="95"/>
+</segment>
+<segment>
+<pinref part="U$2" gate="G$1" pin="SI"/>
+<wire x1="149.86" y1="40.64" x2="162.56" y2="40.64" width="0.1524" layer="91"/>
 </segment>
 </net>
@@
 <label x="35.56" y="10.16" size="1.778" layer="95"/>
 </segment>
+<segment>
+<pinref part="U$2" gate="G$1" pin="SO"/>
+<wire x1="124.46" y1="35.56" x2="114.3" y2="35.56" width="0.1524" layer="91"/>
+</segment>
 </net>
 <net name="D13" class="0">
@@
 <label x="88.9" y="10.16" size="1.778" layer="95"/>
 </segment>
+<segment>
+<pinref part="U$2" gate="G$1" pin="SCK"/>
+<wire x1="124.46" y1="40.64" x2="114.3" y2="40.64" width="0.1524" layer="91"/>
+</segment>
 </net>
